Commit message: 更新代码

File: src/fr5/urdf/fr5.urdf.xacro (robot description, xacro)
@@ -51,10 +51,11 @@
     <axis xyz="0 0 1" />
     <limit lower="-3.14" upper="3.14" effort="1000" velocity="1.0" />
-    <dynamics damping="10.0" friction="10.0"/>
+    <dynamics damping="0.5" friction="0.2"/>
   </joint>
   <link name="link2">
     <inertial>
       <origin xyz="0 0.2 0" rpy="0 0 0" />
-      <mass value="8.0" /> <inertia ixx="0.2" ixy="0" ixz="0" iyy="0.2" iyz="0" izz="0.2" />
+      <mass value="8.0" />
+      <inertia ixx="0.2" ixy="0" ixz="0" iyy="0.2" iyz="0" izz="0.2" />
     </inertial>
     <visual>
@@ -73,10 +74,11 @@
     <axis xyz="0 0 1" />
     <limit lower="-3.14" upper="3.14" effort="1000" velocity="1.0" />
-    <dynamics damping="20.0" friction="20.0"/>
+    <dynamics damping="1.0" friction="0.5"/>
   </joint>
   <link name="link3">
     <inertial>
       <origin xyz="0 0.2 0" rpy="0 0 0" />
-      <mass value="4.0" /> <inertia ixx="0.1" ixy="0" ixz="0" iyy="0.1" iyz="0" izz="0.1" />
+      <mass value="4.0" />
+      <inertia ixx="0.1" ixy="0" ixz="0" iyy="0.1" iyz="0" izz="0.1" />
     </inertial>
     <visual>
@@ -95,10 +97,11 @@
     <axis xyz="0 0 1" />
     <limit lower="-3.14" upper="3.14" effort="1000" velocity="1.0" />
-    <dynamics damping="10.0" friction="10.0"/>
+    <dynamics damping="0.5" friction="0.2"/>
   </joint>
   <link name="link4">
     <inertial>
       <origin xyz="0 0 0" rpy="0 0 0" />
-      <mass value="1.5" /> <inertia ixx="0.05" ixy="0" ixz="0" iyy="0.05" iyz="0" izz="0.05" />
+      <mass value="1.5" />
+      <inertia ixx="0.05" ixy="0" ixz="0" iyy="0.05" iyz="0" izz="0.05" />
     </inertial>
     <visual>
@@ -117,10 +120,11 @@
     <axis xyz="0 0 1" />
     <limit lower="-3.14" upper="3.14" effort="500" velocity="1.0" />
-    <dynamics damping="5.0" friction="5.0"/>
+    <dynamics damping="0.3" friction="0.1"/>
   </joint>
   <link name="link5">
     <inertial>
       <origin xyz="0 0 0" rpy="0 0 0" />
-      <mass value="1.5" /> <inertia ixx="0.05" ixy="0" ixz="0" iyy="0.05" iyz="0" izz="0.05" />
+      <mass value="1.5" />
+      <inertia ixx="0.05" ixy="0" ixz="0" iyy="0.05" iyz="0" izz="0.05" />
     </inertial>
     <visual>
@@ -137,12 +141,13 @@
     <origin xyz="6.5538E-05 0.1018 0" rpy="1.5708 0 0" />
     <parent link="link4" /><child link="link5" />
-    <axis xyz="-0.00064375 0 1" />
+    <axis xyz="0 0 1" />
     <limit lower="-3.14" upper="3.14" effort="500" velocity="1.0" />
-    <dynamics damping="5.0" friction="5.0"/>
+    <dynamics damping="0.3" friction="0.1"/>
   </joint>
   <link name="link6">
     <inertial>
       <origin xyz="0 0 -0.01" rpy="0 0 0" />
-      <mass value="0.5" /> <inertia ixx="0.01" ixy="0" ixz="0" iyy="0.01" iyz="0" izz="0.01" />
+      <mass value="0.5" />
+      <inertia ixx="0.01" ixy="0" ixz="0" iyy="0.01" iyz="0" izz="0.01" />
     </inertial>
     <visual>
@@ -159,7 +164,7 @@
     <origin xyz="0.0998 0 6.4246E-05" rpy="-1.5708 0 -1.5708" />
     <parent link="link5" /><child link="link6" />
-    <axis xyz="0 -0.00064375 1" />
+    <axis xyz="0 0 1" />
     <limit lower="-3.14" upper="3.14" effort="500" velocity="1.0" />
-    <dynamics damping="2.0" friction="1.0"/>
+    <dynamics damping="0.2" friction="0.1"/>
   </joint>
   <link name="tool0"/>
@@ -171,9 +176,10 @@
   <xacro:macro name="fr5_ros2_control_joint" params="joint_name">
     <joint name="${joint_name}">
-      <command_interface name="effort"/>
+      <command_interface name="position"/>
       <state_interface name="position">
         <param name="initial_value">0.0</param>
       </state_interface>
       <state_interface name="velocity"/>
+      <state_interface name="effort"/>
     </joint>
   </xacro:macro>
@@ -189,10 +195,17 @@
     <xacro:fr5_ros2_control_joint joint_name="joint6"/>
     <joint name="left_finger_joint">
-      <command_interface name="position"/> <state_interface name="position"><param name="initial_value">0.0</param></state_interface>
+      <command_interface name="position"/>
+      <state_interface name="position">
+        <param name="initial_value">0.0</param>
+      </state_interface>
       <state_interface name="velocity"/>
+      <state_interface name="effort"/>
     </joint>
     <joint name="right_finger_joint">
-      <state_interface name="position"><param name="initial_value">0.0</param></state_interface>
+      <state_interface name="position">
+        <param name="initial_value">0.0</param>
+      </state_interface>
       <state_interface name="velocity"/>
+      <state_interface name="effort"/>
     </joint>
   </ros2_control>
@@ -202,4 +215,5 @@
       <robot_param_node>robot_state_publisher</robot_param_node>
       <parameters>$(find fr5)/config/fr5_controllers.yaml</parameters>
+      <update_rate>100</update_rate>
     </plugin>
     <plugin filename="libgazebo_ros_mimic_joint_plugin.so" name="mimic_joint_plugin">

File: src/robot_fr5_moveit_config/config/fr5.urdf.xacro (robot description, xacro)
@@ -51,10 +51,12 @@
     <axis xyz="0 0 1" />
     <limit lower="-3.14" upper="3.14" effort="1000" velocity="1.0" />
-    <dynamics damping="10.0" friction="10.0"/>
+    <!-- 降低阻尼/摩擦到合理范围（0.1-1.0） -->
+    <dynamics damping="0.5" friction="0.2"/>
   </joint>
   <link name="link2">
     <inertial>
       <origin xyz="0 0.2 0" rpy="0 0 0" />
-      <mass value="8.0" /> <inertia ixx="0.2" ixy="0" ixz="0" iyy="0.2" iyz="0" izz="0.2" />
+      <mass value="8.0" />
+      <inertia ixx="0.2" ixy="0" ixz="0" iyy="0.2" iyz="0" izz="0.2" />
     </inertial>
     <visual>
@@ -73,10 +75,11 @@
     <axis xyz="0 0 1" />
     <limit lower="-3.14" upper="3.14" effort="1000" velocity="1.0" />
-    <dynamics damping="20.0" friction="20.0"/>
+    <dynamics damping="1.0" friction="0.5"/>
   </joint>
   <link name="link3">
     <inertial>
       <origin xyz="0 0.2 0" rpy="0 0 0" />
-      <mass value="4.0" /> <inertia ixx="0.1" ixy="0" ixz="0" iyy="0.1" iyz="0" izz="0.1" />
+      <mass value="4.0" />
+      <inertia ixx="0.1" ixy="0" ixz="0" iyy="0.1" iyz="0" izz="0.1" />
     </inertial>
     <visual>
@@ -95,10 +98,11 @@
     <axis xyz="0 0 1" />
     <limit lower="-3.14" upper="3.14" effort="1000" velocity="1.0" />
-    <dynamics damping="10.0" friction="10.0"/>
+    <dynamics damping="0.5" friction="0.2"/>
   </joint>
   <link name="link4">
     <inertial>
       <origin xyz="0 0 0" rpy="0 0 0" />
-      <mass value="1.5" /> <inertia ixx="0.05" ixy="0" ixz="0" iyy="0.05" iyz="0" izz="0.05" />
+      <mass value="1.5" />
+      <inertia ixx="0.05" ixy="0" ixz="0" iyy="0.05" iyz="0" izz="0.05" />
     </inertial>
     <visual>
@@ -117,10 +121,11 @@
     <axis xyz="0 0 1" />
     <limit lower="-3.14" upper="3.14" effort="500" velocity="1.0" />
-    <dynamics damping="5.0" friction="5.0"/>
+    <dynamics damping="0.3" friction="0.1"/>
   </joint>
   <link name="link5">
     <inertial>
       <origin xyz="0 0 0" rpy="0 0 0" />
-      <mass value="1.5" /> <inertia ixx="0.05" ixy="0" ixz="0" iyy="0.05" iyz="0" izz="0.05" />
+      <mass value="1.5" />
+      <inertia ixx="0.05" ixy="0" ixz="0" iyy="0.05" iyz="0" izz="0.05" />
     </inertial>
     <visual>
@@ -137,12 +142,14 @@
     <origin xyz="6.5538E-05 0.1018 0" rpy="1.5708 0 0" />
     <parent link="link4" /><child link="link5" />
-    <axis xyz="-0.00064375 0 1" />
+    <!-- 修正 axis 为精确值，避免微小小数引发精度问题 -->
+    <axis xyz="0 0 1" />
     <limit lower="-3.14" upper="3.14" effort="500" velocity="1.0" />
-    <dynamics damping="5.0" friction="5.0"/>
+    <dynamics damping="0.3" friction="0.1"/>
   </joint>
   <link name="link6">
     <inertial>
       <origin xyz="0 0 -0.01" rpy="0 0 0" />
-      <mass value="0.5" /> <inertia ixx="0.01" ixy="0" ixz="0" iyy="0.01" iyz="0" izz="0.01" />
+      <mass value="0.5" />
+      <inertia ixx="0.01" ixy="0" ixz="0" iyy="0.01" iyz="0" izz="0.01" />
     </inertial>
     <visual>
@@ -159,7 +166,8 @@
     <origin xyz="0.0998 0 6.4246E-05" rpy="-1.5708 0 -1.5708" />
     <parent link="link5" /><child link="link6" />
-    <axis xyz="0 -0.00064375 1" />
+    <!-- 修正 axis 为精确值 -->
+    <axis xyz="0 0 1" />
     <limit lower="-3.14" upper="3.14" effort="500" velocity="1.0" />
-    <dynamics damping="2.0" friction="1.0"/>
+    <dynamics damping="0.2" friction="0.1"/>
   </joint>
   <link name="tool0"/>
@@ -169,4 +177,5 @@
     <child link="tool0" />
   </joint>
+  <!-- 完善 ros2_control 关节配置 -->
   <xacro:macro name="fr5_ros2_control_joint" params="joint_name">
     <joint name="${joint_name}">
@@ -176,4 +185,5 @@
       </state_interface>
       <state_interface name="velocity"/>
+      <state_interface name="effort"/>
     </joint>
   </xacro:macro>
@@ -188,11 +198,19 @@
     <xacro:fr5_ros2_control_joint joint_name="joint5"/>
     <xacro:fr5_ros2_control_joint joint_name="joint6"/>
+    <!-- 完善夹爪关节的 control 配置 -->
     <joint name="left_finger_joint">
-      <command_interface name="position"/> <state_interface name="position"><param name="initial_value">0.0</param></state_interface>
+      <command_interface name="position"/>
+      <state_interface name="position">
+        <param name="initial_value">0.0</param>
+      </state_interface>
       <state_interface name="velocity"/>
+      <state_interface name="effort"/>
     </joint>
     <joint name="right_finger_joint">
-      <state_interface name="position"><param name="initial_value">0.0</param></state_interface>
+      <state_interface name="position">
+        <param name="initial_value">0.0</param>
+      </state_interface>
       <state_interface name="velocity"/>
+      <state_interface name="effort"/>
     </joint>
   </ros2_control>
@@ -202,4 +220,6 @@
       <robot_param_node>robot_state_publisher</robot_param_node>
       <parameters>$(find fr5)/config/fr5_controllers.yaml</parameters>
+      <!-- 增加超时配置，避免加载等待过久 -->
+      <update_rate>100</update_rate>
     </plugin>
     <plugin filename="libgazebo_ros_mimic_joint_plugin.so" name="mimic_joint_plugin">

Commit message: 更新机械臂抓取演示代码

File: src/fr5/urdf/fr5.urdf.xacro (robot description, xacro)
@@ -203,4 +203,5 @@
     </joint>
     <joint name="right_finger_joint">
+      <command_interface name="position"/>
       <state_interface name="position">
         <param name="initial_value">0.0</param>
@@ -217,12 +218,20 @@
       <update_rate>100</update_rate>
     </plugin>
-    <plugin filename="libgazebo_ros_mimic_joint_plugin.so" name="mimic_joint_plugin">
-      <joint>left_finger_joint</joint>
-      <mimicJoint>right_finger_joint</mimicJoint>
-      <multiplier>1.0</multiplier>
-      <offset>0.0</offset>
-      <sensitivity>0.0</sensitivity>
-      <maxEffort>200.0</maxEffort>
-      <pid>50.0 0.0 0.1</pid>
+  </gazebo>
+  <gazebo>
+    <plugin name="gazebo_grasp_fix" filename="libgazebo_grasp_fix.so">
+      <arm>
+        <arm_name>fr5_arm</arm_name>
+        <palm_link>link6</palm_link>
+        <gripper_link>left_finger_link</gripper_link>
+        <gripper_link>right_finger_link</gripper_link>
+      </arm>
+      <forces_angle_tolerance>170</forces_angle_tolerance>
+      <update_rate>70</update_rate>
+      <grip_count_threshold>2</grip_count_threshold>
+      <max_grip_count>3</max_grip_count>
+      <release_tolerance>0.005</release_tolerance>
+      <disable_collisions_on_attach>false</disable_collisions_on_attach>
+      <contact_topic>__default_topic__</contact_topic>
     </plugin>
   </gazebo>

File: src/fr5/urdf/simple_gripper.xacro (robot description, xacro)
@@ -56,5 +56,4 @@
       <child link="${prefix}right_finger_link"/>
       <axis xyz="0 -1 0"/>
-      <mimic joint="${prefix}left_finger_joint" multiplier="1" offset="0"/>
       <limit lower="0.0" upper="0.04" effort="60.0" velocity="0.5"/>
       <dynamics damping="1.0" friction="0.1"/>
@@ -81,34 +80,13 @@
     </link>
     <gazebo reference="${prefix}left_finger_link">
-      <mu1>1000.0</mu1>
-      <mu2>1000.0</mu2>
-      <kp>1000000.0</kp>
-      <kd>1.0</kd>
+      <mu1>100000.0</mu1>      <mu2>100000.0</mu2>      <kp>10000.0</kp>         <kd>1000.0</kd>          <minDepth>0.005</minDepth> <maxVel>0.0</maxVel>       <fdir1>0 0 1</fdir1>       </gazebo>
+    <gazebo reference="${prefix}right_finger_link">
+      <mu1>100000.0</mu1>
+      <mu2>100000.0</mu2>
+      <kp>10000.0</kp>
+      <kd>1000.0</kd>
       <minDepth>0.005</minDepth>
-    </gazebo>
-    <gazebo reference="${prefix}right_finger_link">
-      <mu1>1000.0</mu1>
-      <mu2>1000.0</mu2>
-      <kp>1000000.0</kp>
-      <kd>1.0</kd>
-      <minDepth>0.005</minDepth>
-    </gazebo>
-    <gazebo>
-      <plugin name="gazebo_grasp_fix" filename="libgazebo_grasp_fix.so">
-        <arm>
-          <arm_name>simple_gripper</arm_name>
-          <tol_translate>0.02</tol_translate>
-          <tol_angle>0.05</tol_angle>
-          <grip_count_threshold>2</grip_count_threshold>
-          <release_tolerance>0.005</release_tolerance>
-          <disable_collisions_on_attach>false</disable_collisions_on_attach>
-          <contact_topic>__default_topic__</contact_topic>
-          <forces_angle_tolerance>100</forces_angle_tolerance>
-          <update_rate>50</update_rate>
-          <gripper_link>${prefix}left_finger_link</gripper_link>
-          <gripper_link>${prefix}right_finger_link</gripper_link>
-          <palm_link>${prefix}gripper_base_link</palm_link>
-        </arm>
-      </plugin>
+      <maxVel>0.0</maxVel>
+      <fdir1>0 0 1</fdir1>
     </gazebo>
   </xacro:macro>
